File: PCB/CycleOpsPro300toANTPlus_V1.0.brd (EAGLE design)
At the start: 54.4 x 94 mm, 32 parts, among them Q1 2.5A/30V, U1 MCP73831, U2 AP2112K-3.3V, U4 TPS78223DDCR

Commit message: Updated PCB design and placed order for PCBs
Signed-off-by: Matt W <mwasserman@gmail.com>
Parts:
- moved R10 10.2 mm to (19.6, 45.5)
- moved R11 10.2 mm to (16.5, 45.5)
- moved R5 10.2 mm to (14.0, 45.5)
- moved RESET 8.03 mm to (27.2, 79.8)
- moved POWER 8.03 mm to (17.8, 80.0)
- moved CYCLEOPS 7.62 mm to (17.8, 54.6)
- moved OLCD 7.15 mm to (29.5, 65.0)
Routing:
- net GND: track 0.00 -> 229.8 mm, vias 0 -> 3
- net VCC: track 0.00 -> 165.7 mm, vias 0 -> 2
- net TORQUE_ZERO: track 0.00 -> 97.3 mm, vias 0 -> 2
- net VBUS: track 0.00 -> 91.1 mm, vias 0 -> 5
- net VIN: track 0.00 -> 89.7 mm, vias 0 -> 1
- net N$8: track 0.00 -> 84.1 mm, vias 0 -> 1
- net N$2: track 0.00 -> 83.4 mm, vias 0 -> 1
- net SCL: track 0.00 -> 79.8 mm, vias 0 -> 2
- net SDA: track 0.00 -> 74.6 mm, vias 0 -> 2
- net N$1: track 0.00 -> 74.2 mm, vias 0 -> 3
- net 2.95V: track 0.00 -> 60.3 mm, vias 0 -> 5
- net VBAT: track 0.00 -> 59.4 mm
- net N$6: track 0.00 -> 47.6 mm, vias 0 -> 1
- net TXO: track 0.00 -> 29.1 mm
- net RXI: track 0.00 -> 29.0 mm
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
Commit message: Updated CAD Model. Minor corrections to schematic. Updated BOM Parts List.
Signed-off-by: Matt W <mwasserman@gmail.com>
Parts:
- R2: value 10.0K -> 10K
- U4: value TPS78223DDCR -> TPS78001DDCR
Changed lines of the file:
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@@
 <element name="R1" library="SparkFun-Passives" package="0603-RES" value="2.5K" x="43.307" y="46.736" rot="MR0"/>
 <element name="C1" library="SparkFun-Passives" package="0603-CAP" value="4.7uF" x="37.465" y="46.609" rot="MR0"/>
-<element name="R2" library="SparkFun-Passives" package="0603-RES" value="10.0K" x="43.307" y="44.069" rot="MR0"/>
+<element name="R2" library="SparkFun-Passives" package="0603-RES" value="10K" x="43.307" y="44.069" rot="MR0"/>
 <element name="Q1" library="SparkFun-DiscreteSemi" package="SOT23-3" value="2.5A/30V" x="31.623" y="41.656" rot="MR0">
 <attribute name="PROD_ID" value="TRANS-11308" x="31.623" y="41.656" size="1.778" layer="28" rot="MR0" display="off"/>
@@
 <element name="U$1" library="Networking and WiFI" package="F10644_NRF24AP2" value="F10644_NRF24AP2" x="38.1" y="27.94" rot="R270"/>
 <element name="U$2" library="Molex_Connectors" package="53375-02" value="53375-02" x="6.858" y="43.688" rot="R270"/>
-<element name="U4" library="Texas Instruments_By_element14_Batch_1" package="SOT95P280X110-5N" value="TPS78223DDCR" x="25.4" y="40.386" smashed="yes" rot="MR270">
+<element name="U4" library="Texas Instruments_By_element14_Batch_1" package="SOT95P280X110-5N" value="TPS78001DDCR" x="25.4" y="40.386" smashed="yes" rot="MR270">
 <attribute name="PACKAGE" value="TSOT-23-5" x="25.4" y="40.386" size="1.778" layer="28" rot="MR270" display="off"/>
 <attribute name="OC_FARNELL" value="-" x="25.4" y="40.386" size="1.778" layer="28" rot="MR270" display="off"/>
